File: Filter.kicad_sch (KiCad schematic)
At the start: 7 parts

Commit message: Started Schem.
Parts:
- added J5: 5-1814400-2, sma:518144002, symbol SMA Jacks:5-1814400-2
- L6, L7, L8: footprint (none) -> 0603 Footprint:RESC1608X55N
- VC1, VC2, VC3, VC4: footprint JR100:CAPV_JR100 -> varicaps:CAPV_JR100
Connections:
- net Filter_output: now also J5.1
- net GND: now also J5.2, J5.3, J5.4, J5.5
Other:
- moved on the sheet: L6, L7, L8, VC1, VC2, VC3, VC4

Commit message: Filter Update
Parts:
- J5: value 5-1814400-2 -> 50 ohm; Arrow Part Number 5-1814400-2 -> (none); Arrow Price/Stock https://www.arrow.com/en/products/5-1814400-2/te-connectivi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 -> (none); Height 10.63 -> (none); Link (none) -> https://www.digikey.com/en/products/detail/te-connectivity-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; Manufacturer (none) -> TE Connectivity AMP Connectors; Manufacturer_Name TE Connectivity -> (none); Manufacturer_Part_Number 5-1814400-2 -> (none); Mouser Part Number 571-5-1814400-2 -> (none); Mouser Price/Stock https://www.mouser.co.uk/ProductDetail/TE-Connectivity/5-18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 -> (none); Part Number (none) -> 5-1814400-2; Vendor (none) -> Digikey; Vendor ID (none) -> 17-5-1814400-2CT-ND
- L6, L8: Link (none) -> https://www.digikey.com/en/products/detail/coilcraft/0603DC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; Manufacturer (none) -> Coilcraft; Part Number (none) -> 0603DC-20NXJRW; Vendor (none) -> Digikey; Vendor ID (none) -> 2457-0603DC-20NXJRW-ND
- L7: Link (none) -> https://www.digikey.com/en/products/detail/murata-electroni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; Manufacturer (none) -> Murata Electronics; Part Number (none) -> LQW18AS22NJ0CD; Vendor (none) -> Digikey; Vendor ID (none) -> 490-LQW18AS22NJ0CDCT-ND
- VC1, VC4: footprint varicaps:CAPV_JR100 -> Capacitor_SMD:C_0603_1608Metric_Pad1.08x0.95mm_HandSolder; Availability In Stock -> (none); Check_prices https://www.snapeda.com/parts/JR100/Voltronics/view-part/?r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 -> (none); Link (none) -> https://www.digikey.com/en/products/detail/murata-electroni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; MANUFACTURER Knowles Voltronics -> (none); MAXIMUM_PACKAGE_HEIGHT 1.35mm -> (none); MF Voltronics -> (none); MP JR100 -> (none); Manufacturer (none) -> Murata Electronics; PARTREV 10530 -> (none); Package Voltronics -> (none); Part Number (none) -> GCM1885C2A6R8BA16D; Price None -> (none); Purchase-URL https://www.snapeda.com/api/url_track_click_mouser/?unipart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 -> (none); STANDARD Manufacturer Recommendation -> (none); SnapEDA_Link https://www.snapeda.com/parts/JR100/Voltronics/view-part/?r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 -> (none); Vendor (none) -> Digikey; Vendor ID (none) -> 490-GCM1885C2A6R8BA16DCT-ND
- VC2, VC3: footprint varicaps:CAPV_JR100 -> Capacitor_SMD:C_0603_1608Metric_Pad1.08x0.95mm_HandSolder; Availability In Stock -> (none); Check_prices https://www.snapeda.com/parts/JR100/Voltronics/view-part/?r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 -> (none); Link (none) -> https://www.digikey.com/en/products/detail/murata-electroni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; MANUFACTURER Knowles Voltronics -> (none); MAXIMUM_PACKAGE_HEIGHT 1.35mm -> (none); MF Voltronics -> (none); MP JR100 -> (none); Manufacturer (none) -> Murata Electronics; PARTREV 10530 -> (none); Package Voltronics -> (none); Part Number (none) -> GCM1885C2A120JA16D; Price None -> (none); Purchase-URL https://www.snapeda.com/api/url_track_click_mouser/?unipart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 -> (none); STANDARD Manufacturer Recommendation -> (none); SnapEDA_Link https://www.snapeda.com/parts/JR100/Voltronics/view-part/?r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 -> (none); Vendor (none) -> Digikey; Vendor ID (none) -> 490-8009-1-ND
