File: Main.kicad_pcb (KiCad board)
At the start: 4 copper layers, 69.6 x 40 mm, 49 parts, among them IC1 SKYA21001, IC2 BGA420H6327XTSA1, J1 1935776, J2 Conn_01x06_Pin, J3 Conn_01x04_Pin, J5 5-1814400-2, U1 SX1278, U2 TRF37D73IDSGT, U4 SN74AHC1G14DBVR, U5 SN74AHC1G14DBVR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

Commit message: Filter Update
Parts:
- removed C14: 100 pF, Capacitor_SMD:C_0603_1608Metric_Pad1.08x0.95mm_HandSolder
- added CR1: PESD3V3Y1BSFYL, TVS Diode:SOD962-2_DSN0603-2_NEX-L, F.Cu at (157.1, 87.9)
- added D2: -, 0603 LED:LEDC1608X35N, F.Cu at (149.9, 84.0)
- added F1: 0ZCJ0025AF2E, PTC FUSE:0ZCJ_BEL, F.Cu at (158.9, 84.8)
- added R4: 1k, Resistor_SMD:R_0603_1608Metric_Pad0.98x0.95mm_HandSolder, F.Cu at (149.0, 81.3)
- added REF**: MountingHole_2.7mm_M2.5_ISO7380_Pad, MountingHole:MountingHole_2.7mm_M2.5_ISO7380_Pad, F.Cu at (110.5, 73.5)
- added REF**: MountingHole_2.7mm_M2.5_ISO7380_Pad, MountingHole:MountingHole_2.7mm_M2.5_ISO7380_Pad, F.Cu at (171.5, 112.5)
- added REF**: MountingHole_2.7mm_M2.5_ISO7380_Pad, MountingHole:MountingHole_2.7mm_M2.5_ISO7380_Pad, F.Cu at (171.5, 73.5)
- added REF**: MountingHole_2.7mm_M2.5_ISO7380_Pad, MountingHole:MountingHole_2.7mm_M2.5_ISO7380_Pad, F.Cu at (110.5, 112.5)
- D1: value LTST-C190KRKT -> -
- IC1: value SKYA21001 -> -
- IC2: value BGA420H6327XTSA1 -> -
- J1: value 1935776 -> -
- J2: value Conn_01x06_Pin -> DO NOT PLACE
- J3: value Conn_01x04_Pin -> DO NOT PLACE
- J5: value 5-1814400-2 -> 50 ohm
- S1: value PTS810SJK250SMTRLFS -> -
- U1: value SX1278 -> -
- U2: value TRF37D73IDSGT -> -
- U4, U5: value SN74AHC1G14DBVR -> -
- VC1, VC2, VC3, VC4: footprint varicaps:CAPV_JR100 -> Capacitor_SMD:C_0603_1608Metric_Pad1.08x0.95mm_HandSolder
- Y1: value ASTX-13-D-32.000MHz-I05-T -> 32 MHz
- moved L4 42.0 mm to (145.9, 96.9), turned to 90 degrees
- moved U4 41.8 mm to (114.9, 100.4), turned to 90 degrees
- moved C17 41.5 mm to (144.2, 95.0), turned to 90 degrees
- moved C18 38.8 mm to (141.4, 96.0)
- moved C13 37.2 mm to (129.5, 104.9)
- moved C12 36.9 mm to (125.0, 103.0), turned to 90 degrees
- moved L5 33.9 mm to (131.6, 95.3), turned to 90 degrees
- moved L6 32.8 mm to (151.3, 100.5)
- moved U5 30.8 mm to (119.5, 100.8)
- moved C19 30.8 mm to (129.0, 94.4), turned to 180 degrees
- moved L7 30.6 mm to (156.5, 100.5)
- moved C4 30.6 mm to (120.2, 96.8), turned to 180 degrees
- moved L8 29.4 mm to (161.8, 100.5)
- moved R3 29.0 mm to (154.0, 81.3), turned to 180 degrees
- moved C1 28.8 mm to (114.9, 88.0), turned to 90 degrees
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Connections:
- IC1 pad 5: Net-(IC1-J1) -> Filter_input
- J1 pad 01: +3.3V -> Net-(F1-Pad2)
Routing:
- net GND: track 0.00 -> 68.6 mm, vias 0 -> 52
- net Antenna_State: track 0.00 -> 59.2 mm, vias 0 -> 2
- net +3.3V: track 0.00 -> 37.3 mm, vias 0 -> 13
- net Net-(IC1-V2): track 0.00 -> 36.0 mm, vias 0 -> 2
- net /DIO0: track 0.00 -> 30.6 mm, vias 0 -> 1
- net /DIO1: track 0.00 -> 29.6 mm, vias 0 -> 1
- net Net-(IC1-V1): track 0.00 -> 29.6 mm, vias 0 -> 2
- net /DIO2: track 0.00 -> 29.3 mm, vias 0 -> 1
- net /DIO3: track 0.00 -> 29.0 mm, vias 0 -> 1
- net /DIO4: track 0.00 -> 28.3 mm, vias 0 -> 1
- net /DIO5: track 0.00 -> 27.9 mm, vias 0 -> 1
- net Net-(U1-~{RESET}): track 0.00 -> 25.1 mm
- net Net-(J3-Pin_1): track 0.00 -> 14.2 mm
- net Net-(J3-Pin_4): track 0.00 -> 13.9 mm
- net Net-(J3-Pin_2): track 0.00 -> 13.4 mm
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- added copper zone on In2.Cu, net +3.3V
- added copper zone on B.Cu, net GND
- added copper zone on F.Cu, net GND
- added copper zone on In1.Cu, net GND
Other:
- board size 69.6 x 40 mm -> 69.6 x 46.8 mm
- board text added: "R1"
