File: Main.kicad_sch (KiCad schematic)
At the start: 41 parts, among them IC1 SKYA21001, IC2 BGA420H6327XTSA1, J1 1935776, J2 Conn_01x06_Pin, J3 Conn_01x04_Pin, U1 SX1278, U2 TRF37D73IDSGT, U4 SN74AHC1G14DBVR, U5 SN74AHC1G14DBVR, Y1 ASTX-13-D-32.000MHz-I05-T

Commit message: Started Schem.
Parts:
- D1: footprint LTST-C190KRKT:LEDC1608X35N -> 0603 LED:LEDC1608X35N
- IC1: footprint SOT65P220X110-6N -> skya21001:SOT65P220X110-6N
- IC2: footprint SOT343 -> bga420:SOT343
- J1: footprint 1935776:PHOENIX_1935776 -> terminal block:PHOENIX_1935776
Changed lines of the file:
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@@
     )
   )
-  (global_label "Power_Amp_Out" (shape input) (at 139.7 170.18 0) (fields_autoplaced)
+  (global_label "Power_Amp_Out" (shape input) (at 137.16 170.18 0) (fields_autoplaced)
     (effects (font (size 1.27 1.27)) (justify left))
-    (property "Intersheetrefs" "${INTERSHEET_REFS}" (at 157.3014 170.18 0)
+    (property "Intersheetrefs" "${INTERSHEET_REFS}" (at 154.7614 170.18 0)
       (effects (font (size 1.27 1.27)) (justify left))
     )
@@
       (effects (font (size 1.27 1.27)))
     )
-    (property "Footprint" "SOT65P220X110-6N" (at 255.27 57.785 0)
+    (property "Footprint" "skya21001:SOT65P220X110-6N" (at 255.27 57.785 0)
       (effects (font (size 1.27 1.27)) (justify left) hide)
     )
@@
       (effects (font (size 1.27 1.27)))
     )
-    (property "Footprint" "SOT343" (at 231.14 124.46 0)
+    (property "Footprint" "bga420:SOT343" (at 231.14 124.46 0)
       (effects (font (size 1.27 1.27)) (justify left) hide)
     )
@@
       (effects (font (size 1.27 1.27)) (justify right) hide)
     )
-    (property "Footprint" "LTST-C190KRKT:LEDC1608X35N" (at 238.76 35.56 0)
+    (property "Footprint" "0603 LED:LEDC1608X35N" (at 238.76 35.56 0)
       (effects (font (size 1.27 1.27)) (justify bottom) hide)
     )
@@
       (effects (font (size 1.27 1.27)) (justify left) hide)
     )
-    (property "Footprint" "1935776:PHOENIX_1935776" (at 220.98 36.195 0)
-      (effects (font (size 1.27 1.27)) (justify bottom) hide)
-    )
+    (property "Footprint" "terminal block:PHOENIX_1935776" (at 220.98 36.195 0)
+      (effects (font (size 1.27 1.27)) (justify bottom) hide)
+    )

Commit message: Filter Update
Parts:
- removed C14: 100 pF, Capacitor_SMD:C_0603_1608Metric_Pad1.08x0.95mm_HandSolder, symbol Device:C
- added CR1: PESD3V3Y1BSFYL, TVS Diode:SOD962-2_DSN0603-2_NEX-L, symbol TVS Diode:PESD3V3Y1BSFYL
- added D2: -, 0603 LED:LEDC1608X35N, symbol 0603 LED:LTST-C190KRKT
- added F1: 0ZCJ0025AF2E, PTC FUSE:0ZCJ_BEL, symbol PTC Fuse:0ZCJ0025AF2E
- added R4: 1k, Resistor_SMD:R_0603_1608Metric_Pad0.98x0.95mm_HandSolder, symbol Device:R
- C1, C12, C13: Link (none) -> https://www.digikey.com/en/products/detail/w%C3%BCrth-elekt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; Manufacturer (none) -> Würth Elektronik; Part Number (none) -> 885012106010; Vendor (none) -> Digikey; Vendor ID (none) -> 732-7907-1-ND
- C10, C9: Link (none) -> https://www.digikey.com/en/products/detail/w%C3%BCrth-elekt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; Manufacturer (none) -> Würth Elektronik; Part Number (none) -> 885012006029; Vendor (none) -> Digikey; Vendor ID (none) -> 732-7771-1-ND
- C11: Link (none) -> https://www.digikey.com/en/products/detail/w%C3%BCrth-elekt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; Manufacturer (none) -> Würth Elektronik; Part Number (none) -> 885012006030; Vendor (none) -> Digikey; Vendor ID (none) -> 732-7772-1-ND
- C15, C16, C18, C21: Link (none) -> https://www.digikey.com/en/products/detail/w%C3%BCrth-elekt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; Manufacturer (none) -> Würth Elektronik; Part Number (none) -> 885012006023; Vendor (none) -> Digikey; Vendor ID (none) -> 732-7766-1-ND
- C17, C19: Link (none) -> https://www.digikey.com/en/products/detail/w%C3%BCrth-elekt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; Manufacturer (none) -> Würth Elektronik; Part Number (none) -> 885012006047; Vendor (none) -> Digikey; Vendor ID (none) -> 732-7789-1-ND
- C2, C4, C5, C6: Link (none) -> https://www.digikey.com/en/products/detail/w%C3%BCrth-elekt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; Manufacturer (none) -> Würth Elektronik; Part Number (none) -> 885012206071; Vendor (none) -> Digikey; Vendor ID (none) -> 732-7989-1-ND
- C20: Link (none) -> https://www.digikey.com/en/products/detail/w%C3%BCrth-elekt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; Manufacturer (none) -> Würth Elektronik; Part Number (none) -> 885012006002; Vendor (none) -> Digikey; Vendor ID (none) -> 732-7746-1-ND
- C3: Link (none) -> https://www.digikey.com/en/products/detail/w%C3%BCrth-elekt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; Manufacturer (none) -> Würth Elektronik; Part Number (none) -> 885012106005; Vendor (none) -> Digikey; Vendor ID (none) -> 732-7902-1-ND
- C7: Link (none) -> https://www.digikey.com/en/products/detail/w%C3%BCrth-elekt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; Manufacturer (none) -> Würth Elektronik; Part Number (none) -> 885012006017; Vendor (none) -> Digikey; Vendor ID (none) -> 732-7760-1-ND
- C8: Link (none) -> https://www.digikey.com/en/products/detail/w%C3%BCrth-elekt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; Manufacturer (none) -> Würth Elektronik; Part Number (none) -> 885012006087; Vendor (none) -> Digikey; Vendor ID (none) -> 732-12044-1-ND
- D1: value LTST-C190KRKT -> -; AVAILABILITY In Stock -> (none); Availability In Stock -> (none); Check_prices https://www.snapeda.com/parts/LTST-C190KRKT/Lite-On+Inc./vi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 -> (none); DESCRIPTION Yellow 588nm LED Indication - Discrete 2.1V 0603 (1608 Metr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 -> (none); Link (none) -> https://www.digikey.com/en/products/detail/liteon/LTST-C190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; MF Lite-On Inc. -> (none); MP LTST-C190KRKT -> (none); Manufacturer (none) -> Lite-On Inc.; PACKAGE 0603 Lite-On -> (none); PRICE None -> (none); PURCHASE-URL https://pricing.snapeda.com/search/part/LTST-C190YKT/?ref=e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 -> (none); Package 0603 Lite-On -> (none); Part Number (none) -> LTST-C190KRKT; Price None -> (none); Purchase-URL https://www.snapeda.com/api/url_track_click_mouser/?unipart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 -> (none); SnapEDA_Link https://www.snapeda.com/parts/LTST-C190KRKT/Lite-On+Inc./vi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 -> (none); Vendor (none) -> Digikey; Vendor ID (none) -> 160-1436-1-ND
- IC1: value SKYA21001 -> -; Height 1.1 -> (none); Link (none) -> https://www.digikey.com/en/products/detail/skyworks-solutio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; Manufacturer (none) -> Skyworks Solutions Inc.; Manufacturer_Name Skyworks -> (none); Manufacturer_Part_Number SKYA21001 -> (none); Mouser Part Number 873-SKYA21001 -> (none); Mouser Price/Stock https://www.mouser.co.uk/ProductDetail/Skyworks-Solutions-I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 -> (none); Part Number (none) -> SKYA21001; Vendor (none) -> Digikey; Vendor ID (none) -> 863-1753-1-ND
- IC2: value BGA420H6327XTSA1 -> -; Arrow Part Number BGA420H6327XTSA1 -> (none); Arrow Price/Stock https://www.arrow.com/en/products/bga420h6327xtsa1/infineon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 -> (none); Link (none) -> https://www.digikey.com/en/products/detail/infineon-technol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; Manufacturer (none) -> Infineon Technologies; Manufacturer_Name Infineon -> (none); Manufacturer_Part_Number BGA420H6327XTSA1 -> (none); Mouser Part Number 726-BGA420H6327XTSA1 -> (none); Mouser Price/Stock https://www.mouser.co.uk/ProductDetail/Infineon-Technologie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 -> (none); Part Number (none) -> BGA420H6327XTSA1; Vendor (none) -> Digikey; Vendor ID (none) -> BGA420H6327XTSA1CT-ND
- J1: value 1935776 -> -; AVAILABILITY In Stock -> (none); Availability In Stock -> (none); Check_prices https://www.snapeda.com/parts/1935776/Phoenix+Contact/view-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 -> (none); DESCRIPTION 2 Position Wire to Board Terminal Block Horizontal with Boa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 -> (none); Link (none) -> https://www.digikey.com/en/products/detail/phoenix-contact/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; MF Phoenix Contact -> (none); MP 1935776 -> (none); Manufacturer (none) -> Phoenix Contact; PACKAGE None -> (none); PRICE None -> (none); PURCHASE-URL https://pricing.snapeda.com/search/part/1935776/?ref=eda -> (none); Package None -> (none); Part Number (none) -> 1935776; Price None -> (none); Purchase-URL https://www.snapeda.com/api/url_track_click_mouser/?unipart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 -> (none); SnapEDA_Link https://www.snapeda.com/parts/1935776/Phoenix+Contact/view-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 -> (none); Vendor (none) -> Digikey; Vendor ID (none) -> 277-6405-ND
- J2: value Conn_01x06_Pin -> DO NOT PLACE; Link (none) -> DO NOT PLACE; Manufacturer (none) -> DO NOT PLACE; Part Number (none) -> DO NOT PLACE; Vendor (none) -> DO NOT PLACE; Vendor ID (none) -> DO NOT PLACE
- J3: value Conn_01x04_Pin -> DO NOT PLACE; Link (none) -> DO NOT PLACE; Manufacturer (none) -> DO NOT PLACE; Part Number (none) -> DO NOT PLACE; Vendor (none) -> DO NOT PLACE; Vendor ID (none) -> DO NOT PLACE
- L1, L3: Link (none) -> https://www.digikey.com/en/products/detail/coilcraft/0603DC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; Manufacturer (none) -> Coilcraft; Part Number (none) -> 0603DC-11NXJRW; Vendor (none) -> Digikey; Vendor ID (none) -> 2457-0603DC-11NXJRW-ND
- L2: Link (none) -> https://www.digikey.com/en/products/detail/shenzhen-sunlord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; Manufacturer (none) -> Shenzhen Sunlord Electronics Co., Ltd.; Part Number (none) -> SDWL1608CP7N2JSTF; Vendor (none) -> Digikey; Vendor ID (none) -> 3442-SDWL1608CP7N2JSTFCT-ND
- L4, L5: Link (none) -> https://www.digikey.com/en/products/detail/shenzhen-sunlord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; Manufacturer (none) -> Shenzhen Sunlord Electronics Co., Ltd.; Part Number (none) -> SDWL1608CP24NJSTF; Vendor (none) -> Digikey; Vendor ID (none) -> 3442-SDWL1608CP24NJSTFCT-ND
- R1: Link (none) -> https://www.digikey.com/en/products/detail/panasonic-electr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; Manufacturer (none) -> Panasonic Electronic Components; Part Number (none) -> ERJ-3GEYJ103V; Vendor (none) -> Digikey; Vendor ID (none) -> P10KGCT-ND
- R2: Link (none) -> https://www.digikey.com/en/products/detail/panasonic-electr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; Manufacturer (none) -> Panasonic Electronic Components; Part Number (none) -> ERJ-3GEYJ472V; Vendor (none) -> Digikey; Vendor ID (none) -> P4.7KGCT-ND
- R3: Link (none) -> https://www.digikey.com/en/products/detail/panasonic-electr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; Manufacturer (none) -> Panasonic Electronic Components; Part Number (none) -> ERJ-3GEYJ102V; Vendor (none) -> Digikey; Vendor ID (none) -> P1.0KGCT-ND
- S1: value PTS810SJK250SMTRLFS -> -; Availability In Stock -> (none); Check_prices https://www.snapeda.com/parts/PTS810%20SJK%20250%20SMTR%20L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 -> (none); DESCRIPTION IP40 Black Button Tactile Switch, SPST-NO 50 mA 3mm Surface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 -> (none); HEIGHT mm -> (none); Link (none) -> https://www.digikey.com/en/products/detail/c-k/PTS810-SJK-2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; MANUFACTURER_NAME C & K COMPONENTS -> (none); MANUFACTURER_PART_NUMBER PTS810SJK250SMTRLFS -> (none); MF C&K -> (none); MP PTS810 SJK 250 SMTR LFS -> (none); Manufacturer (none) -> C&K; Package None -> (none); Part Number (none) -> PTS810 SJK 250 SMTR LFS; Price None -> (none); Purchase-URL https://www.snapeda.com/api/url_track_click_mouser/?unipart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 -> (none); RS_PART_NUMBER 1359396P -> (none); RS_PRICE-STOCK http://uk.rs-online.com/web/p/products/1359396P -> (none); SnapEDA_Link https://www.snapeda.com/parts/PTS810%20SJK%20250%20SMTR%20L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 -> (none); Vendor (none) -> Digikey; Vendor ID (none) -> CKN10503CT-ND
- U1: value SX1278 -> -; Availability Not in stock -> (none); Check_prices https://www.snapeda.com/parts/SX1278/Semtech/view-part/?ref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 -> (none); Link (none) -> https://www.digikey.com/en/products/detail/semtech-corporat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; MANUFACTURER Semtech -> (none); MAXIMUM_PACKAGE_HEIGHT 1.00mm -> (none); MF Semtech -> (none); MP SX1278 -> (none); Manufacturer (none) -> Semtech Corporation; PARTREV 7 -> (none); Package VQFN-28 Semtech Corporation -> (none); Part Number (none) -> SX1278IMLTRT; Price None -> (none); STANDARD IPC-7351B -> (none); SnapEDA_Link https://www.snapeda.com/parts/SX1278/Semtech/view-part/?ref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 -> (none); Vendor (none) -> Digikey; Vendor ID (none) -> SX1278IMLTRTCT-ND
- U2: value TRF37D73IDSGT -> -; Availability In Stock -> (none); Check_prices https://www.snapeda.com/parts/TRF37D73IDSGT/Texas+Instrumen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 -> (none); Link (none) -> https://www.digikey.com/en/products/detail/texas-instrument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; MF Texas Instruments -> (none); MP TRF37D73IDSGT -> (none); Manufacturer (none) -> Texas Instruments; Package WSON-8 Texas Instruments -> (none); Part Number (none) -> TRF37D73IDSGT; Price None -> (none); Purchase-URL https://www.snapeda.com/api/url_track_click_mouser/?unipart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 -> (none); SnapEDA_Link https://www.snapeda.com/parts/TRF37D73IDSGT/Texas+Instrumen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 -> (none); Vendor (none) -> Digikey; Vendor ID (none) -> 296-38827-1-ND
- U4, U5: value SN74AHC1G14DBVR -> -; Link (none) -> https://www.digikey.com/en/products/detail/texas-instrument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; Manufacturer (none) -> Texas Instruments; Part Number (none) -> SN74AHC1G14DBVR; Vendor (none) -> Digikey; Vendor ID (none) -> 296-1092-1-ND
- Y1: value ASTX-13-D-32.000MHz-I05-T -> 32 MHz; Availability In Stock -> (none); Check_prices https://www.snapeda.com/parts/ASTX-13-D-32.000MHZ-I05-T/Abr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 -> (none); Link (none) -> https://www.digikey.com/en/products/detail/jauch-quartz/O-3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; MANUFACTURER Abracon -> (none); MAXIMUM_PACKAGE_HEIGHT 0.80mm -> (none); MF Abracon LLC -> (none); MP ASTX-13-D-32.000MHZ-I05-T -> (none); Manufacturer (none) -> Jauch Quartz; PARTREV 01.27.2017 -> (none); Package None -> (none); Part Number (none) -> O 30,0-JT22S-B-K-3,3-LF; Price None -> (none); Purchase-URL https://www.snapeda.com/api/url_track_click_mouser/?unipart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 -> (none); SNAPEDA_PN ASTX-13-A-16.000MHZ-A20-T -> (none); STANDARD Manufacturer Recommendations -> (none); SnapEDA_Link https://www.snapeda.com/parts/ASTX-13-D-32.000MHZ-I05-T/Abr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 -> (none); Vendor (none) -> Digikey; Vendor ID (none) -> 1908-1040-1-ND
Connections:
- net +3.3V: now also CR1.2, F1.1; no longer J1.01
- net Antenna_State: now also D2.A
- net Filter_input: now also IC1.5 (J1)
- net GND: now also CR1.1, R4.1
- new net: D2.C, R4.2
- new net: F1.2, J1.01
Other:
- note added: "2.5 ms startup*"
- note added: "SX1278"
- note removed: "TRANSIEVER"
- moved on the sheet: J1
